Commit message: teleop

File: urdf/dd_navi.xacro (robot description, xacro)
@@ -265,5 +265,5 @@
     <joint name = "hokuyo_joint" type="fixed">
         <axis xyz = "0 1 0"/>
-        <origin rpy = "0 0 ${pi} " xyz = "${-base_width/2+hokuyo_length/2} 0 -${hokuyo_height}"/>
+        <origin rpy = "0 0 ${pi} " xyz = "${-base_width/2+hokuyo_length/2} 0 ${hokuyo_height/2}"/>
         <parent link = "base_link"/>
         <child link = "hokuyo_link"/>

Commit message: map

File: urdf/dd_navi.xacro (robot description, xacro)
@@ -271,5 +271,5 @@
     <xacro:include filename="$(find dd_sim)/urdf/dd_gazebo_plugins.xacro"/>
     <xacro:include filename="$(find dd_sim)/urdf/camera.gazebo"/>
-    <xacro:include filename="$(find dd_sim)/urdf/hokuyo.xacro"/>
+    <xacro:include filename="$(find dd_sim)/urdf/hokuyo.gazebo"/>
     <gazebo>
         <plugin name="gazebo_ros_control" filename="libgazebo_ros_control.so">

File: urdf/mybot.xacro (robot description, xacro)
@@ -228,5 +228,5 @@
       <origin xyz="0 0 0" rpy="0 0 0"/>
       <geometry>
-        <mesh filename="package://diff_drive_bot/meshes/hokuyo.dae"/>
+        <mesh filename="package://dd_sim/meshes/hokuyo.dae"/>
       </geometry>
     </visual>

Commit message: speech

File: urdf/dd_navi.xacro (robot description, xacro)
@@ -5,5 +5,5 @@
     <xacro:property name="base_length" value="0.16"/>
     <xacro:property name="base_height" value="0.03"/>
-    <xacro:property name="wheel_radius" value="0.06"/>
+    <xacro:property name="wheel_radius" value="0.04"/>
     <xacro:property name="wheel_length" value="0.015"/>
     <xacro:property name="wheel_separation" value="0.15"/>
@@ -265,5 +265,5 @@
     <joint name = "hokuyo_joint" type="fixed">
         <axis xyz = "0 1 0"/>
-        <origin rpy = "0 0 ${pi} " xyz = "${-base_width/2+hokuyo_length/2} 0 ${hokuyo_height/2}"/>
+        <origin rpy = "0 0 ${pi} " xyz = "${-base_width/2+hokuyo_length/2} 0 ${hokuyo_height}"/>
         <parent link = "base_link"/>
         <child link = "hokuyo_link"/>
